Commit message: fix: my_rb1_gazebo/urdf/my_rb1_robot.urdf

File: my_rb1_gazebo/urdf/my_rb1_robot.urdf (robot description, URDF)
Before this commit: robot my_robot, 7 links, 6 joints
Joints:
- joint back_caster_joint: origin xyz=-0.1 0.0 -0.15 rpy=0 0 0 -> xyz=-0.1 0.0 -0.125 rpy=0 0 0
- joint front_caster_joint: origin xyz=0.1 0.0 -0.15 rpy=0 0 0 -> xyz=0.1 0.0 -0.125 rpy=0 0 0
